Commit message: Ankles fixed
Now to modify walking, setStand etc to include tail

File: Model/FootUtahBody.SLDASM.urdf (robot description, URDF)
Before this commit: robot UtahBody.SLDASM, 9 links, 8 joints
Links:
- added link Tail, mass 2.43669066002775; collision mesh filename=BodyWithTail/meshes/Tail.STL; visual mesh filename=BodyWithTail/meshes/Tail.STL
Joints:
- added joint Hips_Tail: type continuous, parent base_link, child Tail, origin xyz=-0.193717960242815 0 0.132 rpy=3.14159265358979 0 3.14159265358979, axis 0 0 1

Commit message: Added joint velocity limits to prevent instability/madness

File: Model/FootUtahBody.SLDASM.urdf (robot description, URDF)
Before this commit: robot UtahBody.SLDASM, 10 links, 9 joints
Joints:
- joint Femur_tibia_L: limit (none) -> effort=300 velocity=0.17453292519943295
- joint Femur_tibia_R: limit (none) -> effort=300 velocity=0.17453292519943295
- joint Hip_femur_L: limit (none) -> effort=300 velocity=0.17453292519943295
- joint Hips_Tail: limit (none) -> effort=300 velocity=0.17453292519943295
- joint Hips_femur_R: limit (none) -> effort=300 velocity=0.17453292519943295
- joint Tarsa_foot_L: limit (none) -> effort=300 velocity=0.17453292519943295
- joint Tarsa_foot_R: limit (none) -> effort=300 velocity=0.17453292519943295
- joint Tibia_tarsa_L: limit (none) -> effort=300 velocity=0.17453292519943295
- joint Tibia_tarsa_R: limit (none) -> effort=300 velocity=0.17453292519943295

Commit message: ZMP in for fitness func
Not fucking helping much like. Gonna try adding it into an earlier, working version

File: Model/FootUtahBody.SLDASM.urdf (robot description, URDF)
Before this commit: robot UtahBody.SLDASM, 10 links, 9 joints
Links:
- link Foot_L: mass 10.834771497095713 -> 20.834771497095713
- link Foot_R: mass 10.834771497095712 -> 20.834771497095712

Commit message: Paused tail motion

File: Model/FootUtahBody.SLDASM.urdf (robot description, URDF)
Before this commit: robot UtahBody.SLDASM, 10 links, 9 joints
Links:
- link base_link: mass 24.9329927506 -> 4.9329927506

Commit message: Mess with URDF masses

File: Model/FootUtahBody.SLDASM.urdf (robot description, URDF)
Before this commit: robot UtahBody.SLDASM, 10 links, 9 joints
Links:
- link Foot_L: mass 20.834771497095713 -> 2.834771497095713
- link Foot_R: mass 20.834771497095712 -> 2.834771497095712

Commit message: Got a real rough solution to play with

File: Model/FootUtahBody.SLDASM.urdf (robot description, URDF)
Before this commit: robot UtahBody.SLDASM, 10 links, 9 joints
Links:
- link Femur_L: mass 1.0956267569314 -> 0.10956267569314
- link Femur_R: mass 1.09562675424786 -> 0.109562675424786
- link Foot_L: mass 2.834771497095713 -> 1.034771497095713
- link Foot_R: mass 2.834771497095712 -> 1.034771497095712
- link Tail: mass 2.43669066002775 -> 0.13669066002775
- link Tarsa_L: mass 0.1015318884241 -> 0.01015318884241
- link Tarsa_R: mass 0.1015318884241 -> 0.01015318884241
- link Tibia_L: mass 0.837833351696081 -> 0.0837833351696081
- link Tibia_R: mass 0.837833381982962 -> 0.0837833381982962
- link base_link: mass 4.9329927506 -> 0.9329927506

Commit message: Added keyboard changing of speed

File: Model/FootUtahBody.SLDASM.urdf (robot description, URDF)
Before this commit: robot UtahBody.SLDASM, 10 links, 9 joints
Joints:
- joint Femur_tibia_L: limit effort=300 velocity=0.17453292519943295 -> effort=2 velocity=0.17453292519943295
- joint Femur_tibia_R: limit effort=300 velocity=0.17453292519943295 -> effort=2 velocity=0.17453292519943295
- joint Hip_femur_L: limit effort=300 velocity=0.17453292519943295 -> effort=2 velocity=0.17453292519943295
- joint Hips_Tail: limit effort=300 velocity=0.17453292519943295 -> effort=2 velocity=0.17453292519943295
- joint Hips_femur_R: limit effort=300 velocity=0.17453292519943295 -> effort=2 velocity=0.17453292519943295
- joint Tarsa_foot_L: limit effort=300 velocity=0.17453292519943295 -> effort=2 velocity=0.17453292519943295
- joint Tarsa_foot_R: limit effort=300 velocity=0.17453292519943295 -> effort=2 velocity=0.17453292519943295
- joint Tibia_tarsa_L: limit effort=300 velocity=0.17453292519943295 -> effort=2 velocity=0.17453292519943295
- joint Tibia_tarsa_R: limit effort=300 velocity=0.17453292519943295 -> effort=2 velocity=0.17453292519943295

Commit message: Current

File: Model/FootUtahBody.SLDASM.urdf (robot description, URDF)
Before this commit: robot UtahBody.SLDASM, 10 links, 9 joints
Joints:
- joint Tarsa_foot_L: limit effort=2 velocity=0.17453292519943295 -> effort=20 velocity=0.17453292519943295
- joint Tarsa_foot_R: limit effort=2 velocity=0.17453292519943295 -> effort=20 velocity=0.17453292519943295
